File: PCB/Polyglot-Keyboard.kicad_pcb (KiCad board)
At the start: 2 copper layers, 248 x 76.3 mm, 89 parts, among them SW1 SW_Push, SW10 SW_Push, SW11 SW_Push, SW12 SW_Push, SW13 SW_Push, SW14 SW_Push, SW15 SW_Push, SW16 SW_Push, SW17 SW_Push, SW18 SW_Push, SW19 SW_Push, SW2 SW_Push, SW20 SW_Push, SW21 SW_Push, SW22 SW_Push, SW23 SW_Push, SW24 SW_Push, SW25 SW_Push, SW26 SW_Push, SW27 SW_Push, SW28 SW_Push, SW29 SW_Push, SW3 SW_Push, SW30 SW_Push, SW31 SW_Push, SW32 SW_Push, SW33 SW_Push, SW34 SW_Push, SW35 SW_Push, SW36 SW_Push, SW37 SW_Push, SW38 SW_Push, SW39 SW_Push, SW4 SW_Push, SW40 SW_Push, SW41 SW_Push, SW42 SW_Push, SW5 SW_Push, SW6 SW_Push, SW7 SW_Push, SW8 SW_Push, SW9 SW_Push, U1 RP2040-ZERO

Commit message: Add some images
Parts:
- removed the G*** at (148.8, 114.9)
- added G***: LOGO, Polyglot_footprints:20mm_Sabhya, F.Cu at (70.3, 122.8)
- added G***: LOGO, Polyglot_footprints:20mm_Sabhya, F.Cu at (37.6, 122.7)
- added G***: LOGO, Polyglot_footprints:20mm_Sabhya, F.Cu at (229.0, 121.5)
- added G***: LOGO, Polyglot_footprints:40mm_Sabhya, F.Cu at (149.3, 108.5)
- added G***: LOGO, Polyglot_footprints:20mm_Sabhya, F.Cu at (260.2, 121.7)
- moved H3 9.50 mm to (148.8, 82.8)
- moved D18 1.28 mm to (138.0, 87.8)
- moved D30 1.28 mm to (138.0, 106.8)
- moved D39 1.28 mm to (138.0, 125.9)
Connections:
- U1 pad 10: /COL9 -> /COL8
- U1 pad 11: /COL10 -> /COL7
- U1 pad 12: /COL11 -> /COL6
- U1 pad 7: /COL6 -> /COL11
- U1 pad 8: /COL7 -> /COL10
- U1 pad 9: /COL8 -> /COL9
Routing:
- net /ROW0: track 264.8 -> 240.1 mm, vias 13 -> 0
- net /COL7: track 83.2 -> 107.2 mm, vias 4 -> 0
- net /COL6: track 64.5 -> 85.9 mm, vias 5 -> 0
- net /COL8: track 107.5 -> 124.0 mm, vias 8 -> 0
- net /COL9: track 109.2 -> 120.7 mm, vias 4 -> 0
- net /COL3: track 140.2 -> 130.8 mm
- net /COL10: track 129.8 -> 137.8 mm, vias 4 -> 0
- net /ROW2: track 266.7 -> 259.1 mm, vias 9 -> 0
- net /COL0: track 170.7 -> 166.1 mm, vias 3 -> 0
- net /COL4: track 115.0 -> 110.4 mm, vias 5 -> 0
- net /COL1: track 154.5 -> 151.8 mm, vias 2 -> 0
- net /ROW3: track 166.4 -> 168.3 mm
- net Net-(D30-A): track 7.62 -> 6.23 mm
- net Net-(D18-A): track 7.63 -> 6.24 mm
- net Net-(D39-A): track 7.60 -> 6.23 mm
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
Commit message: Add case files and fix PCB
Parts:
- added G***: LOGO, Polyglot_footprints:20mm_Sabhya, F.Cu at (70.3, 118.3)
- added G***: LOGO, Polyglot_footprints:20mm_Sabhya, F.Cu at (260.2, 118.0)
- added G***: LOGO, Polyglot_footprints:20mm_Sabhya, F.Cu at (229.0, 118.0)
- added G***: LOGO, Polyglot_footprints:20mm_Sabhya, F.Cu at (37.6, 118.2)
- U1: footprint RP2040 Zero:MODULE_RP2040-ZERO -> Polyglot_footprints:MODULE_RP2040-ZERO
- moved D6 13.3 mm to (125.9, 74.4), turned to 0 degrees
- moved G*** 4.90 mm to (229.0, 126.4)
- moved G*** 4.80 mm to (260.2, 126.5)
- moved G*** 3.69 mm to (37.6, 126.3)
- moved G*** 3.32 mm to (70.3, 126.2)
- moved H3 0.17 mm to (148.8, 82.6)
Routing:
- net /ROW0: track 240.1 -> 267.6 mm
- net /ROW3: track 168.3 -> 180.3 mm
- net /ROW2: track 259.1 -> 268.5 mm
- net Net-(D6-A): track 6.23 -> 15.1 mm
- net /COL5: track 91.9 -> 99.7 mm
- net /COL4: track 110.4 -> 116.0 mm
- net /ROW1: track 240.2 -> 243.6 mm
- net /COL6: track 85.9 -> 89.3 mm
- net /COL3: track 130.8 -> 133.3 mm
- net /COL1: track 151.8 -> 149.3 mm
- net /COL7: track 107.2 -> 109.6 mm
- net /COL0: track 166.1 -> 167.7 mm
- net /COL8: track 124.0 -> 124.8 mm
- net Net-(D1-A): vias 0 -> 1
