File: PCB/Polyglot-Keyboard.kicad_sch (KiCad schematic)
At the start: 88 parts, among them SW1 SW_Push, SW10 SW_Push, SW11 SW_Push, SW12 SW_Push, SW13 SW_Push, SW14 SW_Push, SW15 SW_Push, SW16 SW_Push, SW17 SW_Push, SW18 SW_Push, SW19 SW_Push, SW2 SW_Push, SW20 SW_Push, SW21 SW_Push, SW22 SW_Push, SW23 SW_Push, SW24 SW_Push, SW25 SW_Push, SW26 SW_Push, SW27 SW_Push, SW28 SW_Push, SW29 SW_Push, SW3 SW_Push, SW30 SW_Push, SW31 SW_Push, SW32 SW_Push, SW33 SW_Push, SW34 SW_Push, SW35 SW_Push, SW36 SW_Push, SW37 SW_Push, SW38 SW_Push, SW39 SW_Push, SW4 SW_Push, SW40 SW_Push, SW41 SW_Push, SW42 SW_Push, SW5 SW_Push, SW6 SW_Push, SW7 SW_Push, SW8 SW_Push, SW9 SW_Push, U1 RP2040-ZERO

Commit message: Add some images
Connections:
- net COL10: now also U1.8 (GP7); no longer U1.11 (GP10)
- net COL11: now also U1.7 (GP6); no longer U1.12 (GP11)
- net COL6: now also U1.12 (GP11); no longer U1.7 (GP6)
- net COL7: now also U1.11 (GP10); no longer U1.8 (GP7)
- net COL8: now also U1.10 (GP9); no longer U1.9 (GP8)
- net COL9: now also U1.9 (GP8); no longer U1.10 (GP9)

Commit message: Add Firmware
Parts:
- U1: footprint RP2040 Zero:MODULE_RP2040-ZERO -> Polyglot_footprints:MODULE_RP2040-ZERO
Changed lines of the file:
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@@
 			)
 		)
-		(property "Footprint" "RP2040 Zero:MODULE_RP2040-ZERO"
+		(property "Footprint" "Polyglot_footprints:MODULE_RP2040-ZERO"
 			(at 149.86 151.13 0)
 			(hide yes)
